File: hw-module-xesc.kicad_sch (KiCad schematic)
At the start: 51 parts, among them J18 Conn_01x05, J22 Screw_Terminal_01x03, J36 Conn_02x03_Odd_Even, J39 Screw_Terminal_01x02, J42 Conn_01x02, U18 2.54mm 2x2 socket, U21 2.54mm 2x2 socket, U24 2.54mm 2x2 socket, U28 LV2862XDDC, U30 2.54mm 1x6 socket, U33 2.54mm 1x6 socket, U36 2.54mm 1x9 socket, U39 2.54mm 1x5 socket, U8 xESC2

Commit message: Reduce MLCC count (Fixes: #1)
Parts:
- C51, C54, C61, C66, C85, C88, C91, C94: now not fitted
Changed lines of the file:
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@@
 		(in_bom yes)
 		(on_board yes)
-		(dnp no)
+		(dnp yes)
 		(fields_autoplaced yes)
 		(property "Reference" "C61"
@@
 		(in_bom yes)
 		(on_board yes)
-		(dnp no)
+		(dnp yes)
 		(fields_autoplaced yes)
 		(property "Reference" "C88"
@@
 		(in_bom yes)
 		(on_board yes)
-		(dnp no)
+		(dnp yes)
 		(fields_autoplaced yes)
 		(property "Reference" "C85"
@@
 		(in_bom yes)
 		(on_board yes)
-		(dnp no)
+		(dnp yes)
 		(fields_autoplaced yes)
 		(property "Reference" "C91"
@@
 		(in_bom yes)
 		(on_board yes)
-		(dnp no)
+		(dnp yes)
 		(fields_autoplaced yes)
 		(property "Reference" "C51"
@@
 		(in_bom yes)
 		(on_board yes)
-		(dnp no)
+		(dnp yes)
 		(fields_autoplaced yes)
 		(property "Reference" "C66"
@@
 		(in_bom yes)
 		(on_board yes)
-		(dnp no)
+		(dnp yes)
 		(fields_autoplaced yes)
 		(property "Reference" "C94"
@@
 		(in_bom yes)
 		(on_board yes)
-		(dnp no)
+		(dnp yes)
 		(fields_autoplaced yes)
 		(property "Reference" "C54"

Commit message: Updated Capacitors
Parts:
- removed C35: 22uF/25V, Capacitor_SMD:C_0805_2012Metric, symbol Device:C
- added C2: 22uF/6.3V, Capacitor_SMD:C_0603_1608Metric, symbol Device:C
- C21: value 22uF/25V -> 22uF/6.3V; footprint Capacitor_SMD:C_0805_2012Metric -> Capacitor_SMD:C_0603_1608Metric; JLC C45783 -> C59461
Connections:
- net 5V: now also C2.1
- net GND: now also C2.2
